File: pcb/xmasstar.kicad_sch (KiCad schematic)
At the start: 23 parts, among them J1 Conn_01x03, J2 Conn_01x03, J3 Conn_02x04_Odd_Even, J4 Conn_01x03, J5 Conn_01x03, J6 Conn_01x03, J7 Conn_01x03, U1 RT9167A-xxxB

Commit message: Move custom footprints into custom xmasstar library
Parts:
- D1, D10, D11, D2, D3, D4, D5, D6, D7, D8, D9: footprint wirmo_power:1615RGBC -> xmasstar:1615RGBC
- J1, J2, J4, J5, J6, J7: footprint wirmo_power:star_edge -> xmasstar:star_edge
- J3: footprint wirmo_power:02x04_smd -> xmasstar:02x04_smd
Changed lines of the file:
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@@
       (effects (font (size 1.27 1.27)))
     )
-    (property "Footprint" "wirmo_power:1615RGBC" (at 177.8 43.815 0)
+    (property "Footprint" "xmasstar:1615RGBC" (at 177.8 43.815 0)
       (effects (font (size 1.27 1.27)) (justify left top) hide)
     )
@@
       (effects (font (size 1.27 1.27)))
     )
-    (property "Footprint" "wirmo_power:1615RGBC" (at 238.76 43.815 0)
+    (property "Footprint" "xmasstar:1615RGBC" (at 238.76 43.815 0)
       (effects (font (size 1.27 1.27)) (justify left top) hide)
     )
@@
       (effects (font (size 1.27 1.27)))
     )
-    (property "Footprint" "wirmo_power:star_edge" (at 29.845 33.655 0)
+    (property "Footprint" "xmasstar:star_edge" (at 29.845 33.655 0)
       (effects (font (size 1.27 1.27)) hide)
     )
@@
       (effects (font (size 1.27 1.27)) (justify left))
     )
-    (property "Footprint" "wirmo_power:star_edge" (at 265.43 36.195 0)
+    (property "Footprint" "xmasstar:star_edge" (at 265.43 36.195 0)
       (effects (font (size 1.27 1.27)) hide)
     )
@@
       (effects (font (size 1.27 1.27)))
     )
-    (property "Footprint" "wirmo_power:1615RGBC" (at 43.815 41.275 0)
+    (property "Footprint" "xmasstar:1615RGBC" (at 43.815 41.275 0)
       (effects (font (size 1.27 1.27)) (justify left top) hide)
     )
@@
       (effects (font (size 1.27 1.27)))
     )
-    (property "Footprint" "wirmo_power:star_edge" (at 116.84 36.195 0)
+    (property "Footprint" "xmasstar:star_edge" (at 116.84 36.195 0)
       (effects (font (size 1.27 1.27)) hide)
     )
@@
       (effects (font (size 1.27 1.27)))
     )
-    (property "Footprint" "wirmo_power:1615RGBC" (at 147.32 43.815 0)
+    (property "Footprint" "xmasstar:1615RGBC" (at 147.32 43.815 0)
       (effects (font (size 1.27 1.27)) (justify left top) hide)
     )
@@
       (effects (font (size 1.27 1.27)))
     )
-    (property "Footprint" "wirmo_power:1615RGBC" (at 223.52 43.815 0)
+    (property "Footprint" "xmasstar:1615RGBC" (at 223.52 43.815 0)
       (effects (font (size 1.27 1.27)) (justify left top) hide)
     )
@@
       (effects (font (size 1.27 1.27)))
     )
-    (property "Footprint" "wirmo_power:1615RGBC" (at 132.08 43.815 0)
+    (property "Footprint" "xmasstar:1615RGBC" (at 132.08 43.815 0)
       (effects (font (size 1.27 1.27)) (justify left top) hide)
     )
@@
       (effects (font (size 1.27 1.27)))
     )
-    (property "Footprint" "wirmo_power:1615RGBC" (at 162.56 43.815 0)
+    (property "Footprint" "xmasstar:1615RGBC" (at 162.56 43.815 0)
       (effects (font (size 1.27 1.27)) (justify left top) hide)
     )
@@
       (effects (font (size 1.27 1.27)))
     )
-    (property "Footprint" "wirmo_power:1615RGBC" (at 193.04 43.815 0)
+    (property "Footprint" "xmasstar:1615RGBC" (at 193.04 43.815 0)
       (effects (font (size 1.27 1.27)) (justify left top) hide)
     )
@@
       (effects (font (size 1.27 1.27)))
     )
-    (property "Footprint" "wirmo_power:1615RGBC" (at 254 43.815 0)
+    (property "Footprint" "xmasstar:1615RGBC" (at 254 43.815 0)
       (effects (font (size 1.27 1.27)) (justify left top) hide)
     )
@@
       (effects (font (size 1.27 1.27)) (justify left))
     )
-    (property "Footprint" "wirmo_power:star_edge" (at 55.245 33.655 0)
+    (property "Footprint" "xmasstar:star_edge" (at 55.245 33.655 0)
       (effects (font (size 1.27 1.27)) hide)
     )
@@
       (effects (font (size 1.27 1.27)) (justify left))
     )
-    (property "Footprint" "wirmo_power:star_edge" (at 320.675 38.1 0)
+    (property "Footprint" "xmasstar:star_edge" (at 320.675 38.1 0)
       (effects (font (size 1.27 1.27)) hide)
     )
@@
       (effects (font (size 1.27 1.27)))
     )
-    (property "Footprint" "wirmo_power:star_edge" (at 295.275 38.1 0)
+    (property "Footprint" "xmasstar:star_edge" (at 295.275 38.1 0)
       (effects (font (size 1.27 1.27)) hide)
     )
@@
       (effects (font (size 1.27 1.27)))
     )
-    (property "Footprint" "wirmo_power:1615RGBC" (at 208.28 43.815 0)
+    (property "Footprint" "xmasstar:1615RGBC" (at 208.28 43.815 0)
       (effects (font (size 1.27 1.27)) (justify left top) hide)
     )
@@
       (effects (font (size 1.27 1.27)))
     )
-    (property "Footprint" "wirmo_power:1615RGBC" (at 309.245 45.72 0)
+    (property "Footprint" "xmasstar:1615RGBC" (at 309.245 45.72 0)
       (effects (font (size 1.27 1.27)) (justify left top) hide)
     )
@@
       (effects (font (size 1.27 1.27)))
     )
-    (property "Footprint" "wirmo_power:02x04_smd" (at 93.98 34.925 0)
-      (effects (font (size 1.27 1.27)) hide)
-    )
+    (property "Footprint" "xmasstar:02x04_smd" (at 93.98 34.925 0)
+      (effects (font (size 1.27 1.27)) hide)
+    )
